Commit message: fix issues on test

File: urdf/lidar.xacro (robot description, xacro)
@@ -1,79 +1,85 @@
 <?xml version="1.0"?>
 <robot name="ipalidar" xmlns:xacro="http://www.ros.org/wiki/xacro">
-  <link name="world"/>
+  <link name="base_link" />
   <joint name="fixed" type="fixed">
-    <parent link="world"/>
-    <child link="base_link"/>
+    <parent link="base_link" />
+    <child link="laser_base_link" />
   </joint>
   <!-- Base Link -->
-  <link name="base_link">
+  <link name="laser_base_link">
     <collision>
-      <origin xyz="0 0 0" rpy="0 0 0"/>
+      <origin xyz="0 0 0" rpy="0 0 0" />
       <geometry>
-        <box size="0.12 0.12 0.02"/>
+        <box size="0.12 0.12 0.02" />
       </geometry>
     </collision>
     <visual>
-      <origin xyz="0 0 0" rpy="0 0 0"/>
+      <origin xyz="0 0 0" rpy="0 0 0" />
       <geometry>
-        <box size="0.12 0.12 0.02"/>
+        <box size="0.12 0.12 0.02" />
       </geometry>
     </visual>
     <inertial>
-      <mass value="1e-5"/>
-      <origin xyz="0 0 0" rpy="0 0 0"/>
-      <inertia ixx="1e-6" ixy="0" ixz="0" iyy="1e-6" iyz="0" izz="1e-6"/>
+      <mass value="1e-5" />
+      <origin xyz="0 0 0" rpy="0 0 0" />
+      <inertia ixx="1e-6" ixy="0" ixz="0" iyy="1e-6" iyz="0" izz="1e-6" />
     </inertial>
   </link>
   <!-- Lidar itself -->
-  <joint name="hokuyo_joint" type="fixed">
+  <joint name="laser_joint" type="fixed">
     <!-- <axis xyz="0 1 0"/> -->
-    <origin xyz="0 0 0.05" rpy="0 0 0"/>
-    <parent link="base_link"/>
-    <child link="hokuyo_link"/>
+    <origin xyz="0 0 0.05" rpy="0 0 0" />
+    <parent link="laser_base_link" />
+    <child link="laser" />
   </joint>
-  <link name="hokuyo_link">
+  <link name="laser">
     <collision>
-      <origin xyz="0 0 0" rpy="0 0 0"/>
+      <origin xyz="0 0 0" rpy="0 0 0" />
       <geometry>
-        <box size="0.1 0.1 0.1"/>
+        <box size="0.1 0.1 0.1" />
       </geometry>
     </collision>
     <visual>
-      <origin xyz="0 0 0" rpy="0 0 0"/>
+      <origin xyz="0 0 0" rpy="0 0 0" />
       <geometry>
-        <mesh filename="package://better_facto_simuls/meshes/hokuyo.dae"/>
+        <mesh filename="package://better_facto_simuls/meshes/rplidar-a2.stl" />
       </geometry>
     </visual>
     <inertial>
-      <mass value="1e-5"/>
-      <origin xyz="0 0 0" rpy="0 0 0"/>
-      <inertia ixx="1e-6" ixy="0" ixz="0" iyy="1e-6" iyz="0" izz="1e-6"/>
+      <mass value="1e-5" />
+      <origin xyz="0 0 0" rpy="0 0 0" />
+      <inertia ixx="1e-6" ixy="0" ixz="0" iyy="1e-6" iyz="0" izz="1e-6" />
     </inertial>
   </link>
   <!-- Gazebo plugin for ROS -->
-  <gazebo reference="hokuyo_link">
-    <sensor type="ray" name="head_hokuyo_sensor">
-      <pose>0 0 0 0 0 0</pose>
-      <visualize>true</visualize>
+  <!-- RpLidar A2 using CPU -->
+  <gazebo reference="laser">
+    <sensor type="ray" name="head_rplidar_sensor">
+      <pose>0 0 0.06 0 0 0</pose>
+      <visualize>false</visualize>
       <update_rate>40</update_rate>
       <ray>
         <scan>
           <horizontal>
-            <samples>1080</samples>
-            <resolution>0.25</resolution>
-            <min_angle>-3.14</min_angle>
-            <max_angle>3.14</max_angle>
+            <samples>720</samples>
+            <resolution>1</resolution>
+            <min_angle>-3.14159265</min_angle>
+            <max_angle>3.14159265</max_angle>
           </horizontal>
         </scan>
         <range>
-          <min>0.05</min>
-          <max>30.0</max>
+          <min>0.2</min>
+          <max>12.0</max>
           <resolution>0.01</resolution>
         </range>
+        <noise>
+          <type>gaussian</type>
+          <mean>0.0</mean>
+          <stddev>0.01</stddev>
+        </noise>
       </ray>
-      <plugin name="gazebo_ros_head_hokuyo_controller" filename="libgazebo_ros_laser.so">
+      <plugin name="gazebo_ros_head_rplidar_controller" filename="libgazebo_ros_laser.so">
         <topicName>scan</topicName>
-        <frameName>hokuyo_link</frameName>
+        <frameName>laser</frameName>
       </plugin>
     </sensor>
